Commit message: URDF joint mobility testing complete

File: pybullet/learm_description/learm.urdf (robot description, URDF)
Before this commit: robot learm, 12 links, 11 joints
Links:
- removed link finger_left_link
- removed link finger_right_link
- removed link grip_left_link
- removed link grip_right_link
- removed link hand_link
- removed link tendon_left_link
- removed link tendon_right_link
- added link net_link; visual mesh filename=learm_description/net.stl scale=0.01 0.01 0.01
- link base_link: geometry visual mesh filename=learm_description/base.stl scale=10 10 10
- link forearm_link: geometry visual mesh filename=learm_description/forearm.stl scale=10 10 10
- link humerus_link: geometry visual mesh filename=learm_description/humerus.stl scale=10 10 10
- link shoulder_link: geometry visual mesh filename=learm_description/shoulder.stl scale=10 10 10
- link wrist_link: geometry visual mesh filename=learm_description/wrist.stl scale=10 10 10
Joints:
- removed joint elbow
- removed joint finger_left
- removed joint finger_right
- removed joint grip_left
- removed joint grip_right
- removed joint shoulder_lift
- removed joint shoulder_pan
- removed joint tendon_left
- removed joint tendon_right
- removed joint wrist_flex
- removed joint wrist_roll
- added joint base_joint: type revolute, parent base_link, child shoulder_link, origin xyz=0 0 0.59 rpy=0 0 3.14159, axis 0 0 -1, limit lower=-1.57 upper=1.57 effort=1000 velocity=0.5
- added joint elbow_joint: type revolute, parent humerus_link, child forearm_link, origin xyz=0 0 1.05, axis 0 -1 0, limit lower=0 upper=0 effort=1000 velocity=0.5
- added joint net_joint: type fixed, parent wrist_link, child net_link, origin xyz=1.2 0 0.15 rpy=0 0 3.14159
- added joint shoulder_joint: type revolute, parent shoulder_link, child humerus_link, origin xyz=-0.10 0 0.28, axis 0 -1 0, limit lower=0 upper=1.57 effort=1000 velocity=0.5
- added joint wrist_joint: type revolute, parent forearm_link, child wrist_link, origin xyz=0 0 0.90 rpy=0 0 3.14159, axis 0 -1 0, limit lower=0 upper=1.57 effort=1000 velocity=0.5

Commit message: Heuristic controller is looking positive

File: pybullet/learm_description/learm.urdf (robot description, URDF)
Before this commit: robot learm, 6 links, 5 joints
Links:
- link base_link: mass None -> 1.0
- link forearm_link: mass None -> 1.0
- link humerus_link: mass None -> 1.0
- link net_link: mass None -> 1.0
- link shoulder_link: mass None -> 1.0
- link wrist_link: mass None -> 1.0
Joints:
- joint elbow_joint: limit lower=0 upper=0 effort=1000 velocity=0.5 -> lower=0 upper=0 effort=1000 velocity=0
- joint net_joint: origin xyz=1.2 0 0.15 rpy=0 0 3.14159 -> xyz=1.18 0 0.15 rpy=0 0 3.14159
